Commit message: Add portable Orbbec driver and preserve calibration datasets

File: src/fairino16_ctpm2f20_1/config/fairino16_ctpm2f20.urdf (robot description, URDF)
Before this commit: robot fairino16_gripper_robot, 17 links, 16 joints
Links:
- link base_link: geometry collision mesh filename=package://fairino16_ctpm2f20_1/meshes/arm/base_link.STL; visual mesh filename=package://fairino16_ctpm2f20_1/meshes/arm/base_link.STL
- link forearm_link: geometry collision mesh filename=package://fairino16_ctpm2f20_1/meshes/arm/forearm_link.STL; visual mesh filename=package://fairino16_ctpm2f20_1/meshes/arm/forearm_link.STL
- link gripper_base_link: geometry collision mesh filename=package://fairino16_ctpm2f20_1/meshes/visual/base_link.STL; visual mesh filename=package://fairino16_ctpm2f20_1/meshes/visual/base_link.STL
- link gripper_body_link: geometry collision mesh filename=package://fairino16_ctpm2f20_1/meshes/visual/body_link.STL; visual mesh filename=package://fairino16_ctpm2f20_1/meshes/visual/body_link.STL
- link gripper_left_link: geometry collision mesh filename=package://fairino16_ctpm2f20_1/meshes/visual/left_link.STL; visual mesh filename=package://fairino16_ctpm2f20_1/meshes/visual/left_link.STL
- link gripper_right_link: geometry collision mesh filename=package://fairino16_ctpm2f20_1/meshes/visual/right_link.STL; visual mesh filename=package://fairino16_ctpm2f20_1/meshes/visual/right_link.STL
- link shoulder_link: geometry collision mesh filename=package://fairino16_ctpm2f20_1/meshes/arm/shoulder_link.STL; visual mesh filename=package://fairino16_ctpm2f20_1/meshes/arm/shoulder_link.STL
- link upperarm_link: geometry collision mesh filename=package://fairino16_ctpm2f20_1/meshes/arm/upperarm_link.STL; visual mesh filename=package://fairino16_ctpm2f20_1/meshes/arm/upperarm_link.STL
- link wrist1_link: geometry collision mesh filename=package://fairino16_ctpm2f20_1/meshes/arm/wrist1_link.STL; visual mesh filename=package://fairino16_ctpm2f20_1/meshes/arm/wrist1_link.STL
- link wrist2_link: geometry collision mesh filename=package://fairino16_ctpm2f20_1/meshes/arm/wrist2_link.STL; visual mesh filename=package://fairino16_ctpm2f20_1/meshes/arm/wrist2_link.STL
- link wrist3_link: geometry collision mesh filename=package://fairino16_ctpm2f20_1/meshes/arm/wrist3_link.STL; visual mesh filename=package://fairino16_ctpm2f20_1/meshes/arm/wrist3_link.STL
